Commit message: fix urdf coordinate problem

File: urdf/hx300l1.urdf (robot description, URDF)
Before this commit: robot HX300L, 6 links, 5 joints
Links:
- removed link link5
- link base_link: mass 94.155 -> 94.1546039717305; geometry collision mesh filename=package://hx300l/meshes/base_link.STL; visual mesh filename=package://hx300l/meshes/base_link.STL
- link link1: geometry collision mesh filename=package://hx300l/meshes/link1.STL; visual mesh filename=package://hx300l/meshes/link1.STL
- link link2: mass 106.8 -> 132.25; geometry collision mesh filename=package://hx300l/meshes/link2.STL; visual mesh filename=package://hx300l/meshes/link2.STL
- link link3: mass 132.25 -> 52.492850757275; geometry collision mesh filename=package://hx300l/meshes/link3.STL; visual mesh filename=package://hx300l/meshes/link3.STL
- link link4: mass 52.493 -> 18.5659141905672; geometry collision mesh filename=package://hx300l/meshes/link4.STL; visual mesh filename=package://hx300l/meshes/link4.STL
Joints:
- removed joint joint5
- joint joint1: axis 0 0 0 -> 0 0 1; limit (none) -> lower=-2.617 upper=2.617 effort=30 velocity=1.571; type continuous -> revolute
- joint joint2: axis 0 0 0 -> 1 0 0; limit (none) -> lower=-2.617 upper=2.617 effort=30 velocity=1.571; origin xyz=0 0 0 rpy=0 0 0 -> xyz=0 0.3 0.588 rpy=1.5708 1.0519E-30 -6.123E-17; type continuous -> revolute
- joint joint3: axis 0 0 0 -> 0 0 1; limit (none) -> lower=-2.617 upper=2.617 effort=30 velocity=1.571; origin xyz=0 0.3 0.588 rpy=1.5708 1.0519E-30 -6.123E-17 -> xyz=0 1 0 rpy=0 1.5708 0; type continuous -> revolute
- joint joint4: axis 0 0 0 -> 0 1 0; limit (none) -> lower=-2.617 upper=2.617 effort=30 velocity=1.571; origin xyz=0 1 0 rpy=0 1.5708 0 -> xyz=1.8 0.2 0 rpy=-1.5708 0 0; type continuous -> revolute
